Commit message: Rebase from 'upstream'

File: pr2_description/urdf/shoulder_v0/shoulder.urdf.xacro (robot description, xacro)
@@ -3,5 +3,5 @@
 <robot xmlns:sensor="http://playerstage.sourceforge.net/gazebo/xmlschema/#sensor"
        xmlns:controller="http://playerstage.sourceforge.net/gazebo/xmlschema/#controller"
-       xmlns:interface="http://playerstage.sourceforge.net/gazebo/xmlschema/#interface"
+       xmlns:interface="http://ros.org/wiki/xacro"
        xmlns:xacro="http://ros.org/wiki/xacro">
   <!-- Things that are needed only for Gazebo (not the physical robot).  These include
@@ -10,6 +10,6 @@
   <xacro:include filename="$(find pr2_description)/urdf/shoulder_v0/shoulder.transmission.xacro" />
   <xacro:include filename="$(find pr2_description)/urdf/common.xacro" />
-  <property name="shoulder_lift_length" value="0.10" />  <!--TODO Define and give source-->
-  <property name="shoulder_lift_radius" value="0.12" />  <!--TODO Define and give source-->
+  <xacro:property name="shoulder_lift_length" value="0.10" />  <!--TODO Define and give source-->
+  <xacro:property name="shoulder_lift_radius" value="0.12" />  <!--TODO Define and give source-->
  <!-- ============================   Shoulder   ============================ -->
   <xacro:macro name="pr2_shoulder_v0" params="side parent reflect *origin">
@@ -17,5 +17,5 @@
     <joint name="${side}_shoulder_pan_joint" type="revolute">
       <axis xyz="0 0 1" />
-      <insert_block name="origin" /> <!-- transform from parent link to this joint frame -->
+      <xacro:insert_block name="origin" /> <!-- transform from parent link to this joint frame -->
       <parent link="${parent}"/>
       <child link="${side}_shoulder_pan_link"/>
@@ -99,5 +99,5 @@
     <joint name="${side}_upper_arm_roll_joint" type="revolute">
       <axis xyz="1 0 0" />
-      <insert_block name="origin" />
+      <xacro:insert_block name="origin" />
       <parent link="${parent}" />
       <child link="${side}_upper_arm_roll_link"/>

File: pr2_description/urdf/tilting_laser_v0/tilting_laser.urdf.xacro (robot description, xacro)
@@ -2,5 +2,5 @@
 <robot xmlns:sensor="http://playerstage.sourceforge.net/gazebo/xmlschema/#sensor"
        xmlns:controller="http://playerstage.sourceforge.net/gazebo/xmlschema/#controller"
-       xmlns:interface="http://playerstage.sourceforge.net/gazebo/xmlschema/#interface"
+       xmlns:interface="http://ros.org/wiki/xacro"
        xmlns:xacro="http://ros.org/wiki/xacro">
   <xacro:include filename="$(find pr2_description)/urdf/tilting_laser_v0/tilting_laser.gazebo.xacro" />
@@ -14,5 +14,5 @@
       <calibration falling="${laser_calib_ref}" />
       <dynamics damping="0.008" />
-      <insert_block name="origin" />
+      <xacro:insert_block name="origin" />
       <parent link="${parent}"/>
       <child link="${name}_mount_link"/>

File: pr2_description/urdf/torso_v0/torso.urdf.xacro (robot description, xacro)
@@ -2,5 +2,5 @@
 <robot xmlns:sensor="http://playerstage.sourceforge.net/gazebo/xmlschema/#sensor"
        xmlns:controller="http://playerstage.sourceforge.net/gazebo/xmlschema/#controller"
-       xmlns:interface="http://playerstage.sourceforge.net/gazebo/xmlschema/#interface"
+       xmlns:interface="http://ros.org/wiki/xacro"
        xmlns:xacro="http://ros.org/wiki/xacro">
   <xacro:include filename="$(find pr2_description)/urdf/torso_v0/torso.gazebo.xacro" />
@@ -14,5 +14,5 @@
       <calibration falling="0.00475" />
       <dynamics damping="20000.0" />
-      <insert_block name="origin" />
+      <xacro:insert_block name="origin" />
       <parent link="${parent}"/>
       <child link="${name}_link"/>

File: pr2_description/urdf/upper_arm_v0/upper_arm.urdf.xacro (robot description, xacro)
@@ -3,5 +3,5 @@
 <robot xmlns:sensor="http://playerstage.sourceforge.net/gazebo/xmlschema/#sensor"
        xmlns:controller="http://playerstage.sourceforge.net/gazebo/xmlschema/#controller"
-       xmlns:interface="http://playerstage.sourceforge.net/gazebo/xmlschema/#interface"
+       xmlns:interface="http://ros.org/wiki/xacro"
        xmlns:xacro="http://ros.org/wiki/xacro">
   <!-- Things that are needed only for Gazebo (not the physical robot).  These include
@@ -11,22 +11,22 @@
   <xacro:include filename="$(find pr2_description)/urdf/common.xacro" />
   <!-- Inertial properties differ slightly for left vs right arm -->
-  <property name="uar_xyz1" value= "0.21398" />
-  <property name="uar_xyz2" value="-0.01621" />
-  <property name="uar_xyz3" value="-0.00020" />
-  <property name="uar_ixx"  value= "0.01537748957" />
-  <property name="uar_ixy"  value= "0.00375711247" />
-  <property name="uar_ixz"  value="-0.00070852914" />
-  <property name="uar_iyy"  value= "0.07473670440" />
-  <property name="uar_iyz"  value="-0.00017936450" />
-  <property name="uar_izz"  value= "0.07608763307" />
-  <property name="ual_xyz1" value= "0.21405" />
-  <property name="ual_xyz2" value= "0.01658" />
-  <property name="ual_xyz3" value="-0.00057" />
-  <property name="ual_ixx"  value= "0.01530603856" />
-  <property name="ual_ixy"  value="-0.00339324862" />
-  <property name="ual_ixz"  value= "0.00060765455" />
-  <property name="ual_iyy"  value= "0.07473694455" />
-  <property name="ual_iyz"  value="-0.00019953729" />
-  <property name="ual_izz"  value= "0.07601594191" />
+  <xacro:property name="uar_xyz1" value= "0.21398" />
+  <xacro:property name="uar_xyz2" value="-0.01621" />
+  <xacro:property name="uar_xyz3" value="-0.00020" />
+  <xacro:property name="uar_ixx"  value= "0.01537748957" />
+  <xacro:property name="uar_ixy"  value= "0.00375711247" />
+  <xacro:property name="uar_ixz"  value="-0.00070852914" />
+  <xacro:property name="uar_iyy"  value= "0.07473670440" />
+  <xacro:property name="uar_iyz"  value="-0.00017936450" />
+  <xacro:property name="uar_izz"  value= "0.07608763307" />
+  <xacro:property name="ual_xyz1" value= "0.21405" />
+  <xacro:property name="ual_xyz2" value= "0.01658" />
+  <xacro:property name="ual_xyz3" value="-0.00057" />
+  <xacro:property name="ual_ixx"  value= "0.01530603856" />
+  <xacro:property name="ual_ixy"  value="-0.00339324862" />
+  <xacro:property name="ual_ixz"  value= "0.00060765455" />
+  <xacro:property name="ual_iyy"  value= "0.07473694455" />
+  <xacro:property name="ual_iyz"  value="-0.00019953729" />
+  <xacro:property name="ual_izz"  value= "0.07601594191" />
   <!-- ============================   Upper Arm   ============================ -->
   <!-- Includes elbow flex, FA roll joints in macros below -->
