Commit message: Rebase from 'upstream'

File: pr2_description/robots/pr2.urdf.xacro (robot description, xacro)
@@ -1,8 +1,4 @@
 <?xml version="1.0"?>
-<robot xmlns:sensor="http://playerstage.sourceforge.net/gazebo/xmlschema/#sensor"
-       xmlns:controller="http://playerstage.sourceforge.net/gazebo/xmlschema/#controller"
-       xmlns:interface="http://playerstage.sourceforge.net/gazebo/xmlschema/#interface"
-       xmlns:xacro="http://playerstage.sourceforge.net/gazebo/xmlschema/#interface"
-       name="pr2" >
+<robot xmlns:xacro="http://ros.org/wiki/xacro" name="pr2" >
   <!-- The following included files set up definitions of parts of the robot body -->
   <!-- misc common stuff? -->
@@ -123,6 +119,8 @@
   </xacro:wge100_camera_v0>
   <!-- Kinect models -->
+  <xacro:arg name="KINECT1" default="false" />
+  <xacro:arg name="KINECT2" default="false" />
   <!-- Kinect2 xacro -->
-  <xacro:if value="$(optenv KINECT2 false)">
+  <xacro:if value="$(arg KINECT2)">
     <xacro:include filename="$(find pr2_description)/urdf/sensors/kinect2.urdf.xacro" />
     <xacro:kinect2_v0 name="head_mount" parent="head_plate_frame" >
@@ -131,6 +129,6 @@
   </xacro:if>
   <!-- Kinect1 xacro -->
-  <xacro:unless value="$(optenv KINECT2 false)">
-    <xacro:if value="$(optenv KINECT1 false)">
+  <xacro:unless value="$(arg KINECT2)">
+    <xacro:if value="$(arg KINECT1)">
       <xacro:include filename="$(find pr2_description)/urdf/sensors/kinect_prosilica_camera.urdf.xacro" />
       <!-- Base of Kinect/Prosilica Mount -->

File: pr2_description/robots/pr2_no_arms.urdf.xacro (robot description, xacro)
@@ -1,8 +1,4 @@
 <?xml version="1.0"?>
-<robot xmlns:sensor="http://playerstage.sourceforge.net/gazebo/xmlschema/#sensor"
-       xmlns:controller="http://playerstage.sourceforge.net/gazebo/xmlschema/#controller"
-       xmlns:interface="http://playerstage.sourceforge.net/gazebo/xmlschema/#interface"
-       xmlns:xacro="http://playerstage.sourceforge.net/gazebo/xmlschema/#interface"
-       name="pr2" >
+<robot xmlns:xacro="http://ros.org/wiki/xacro" name="pr2" >
   <!-- The following included files set up definitions of parts of the robot body -->
   <!-- misc common stuff? -->

File: pr2_description/robots/pr2_no_kinect.urdf.xacro (robot description, xacro)
@@ -1,8 +1,4 @@
 <?xml version="1.0"?>
-<robot xmlns:sensor="http://playerstage.sourceforge.net/gazebo/xmlschema/#sensor"
-       xmlns:controller="http://playerstage.sourceforge.net/gazebo/xmlschema/#controller"
-       xmlns:interface="http://playerstage.sourceforge.net/gazebo/xmlschema/#interface"
-       xmlns:xacro="http://playerstage.sourceforge.net/gazebo/xmlschema/#interface"
-       name="pr2" >
+<robot xmlns:xacro="http://ros.org/wiki/xacro" name="pr2" >
   <!-- The following included files set up definitions of parts of the robot body -->
   <!-- misc common stuff? -->

File: pr2_description/robots/pr2_se.urdf.xacro (robot description, xacro)
@@ -1,8 +1,4 @@
 <?xml version="1.0"?>
-<robot xmlns:sensor="http://playerstage.sourceforge.net/gazebo/xmlschema/#sensor"
-       xmlns:controller="http://playerstage.sourceforge.net/gazebo/xmlschema/#controller"
-       xmlns:interface="http://playerstage.sourceforge.net/gazebo/xmlschema/#interface"
-       xmlns:xacro="http://playerstage.sourceforge.net/gazebo/xmlschema/#interface"
-       name="pr2" >
+<robot xmlns:xacro="http://ros.org/wiki/xacro" name="pr2" >
   <!-- The following included files set up definitions of parts of the robot body -->
   <!-- misc common stuff? -->

File: pr2_description/urdf/base_v0/base.transmission.xacro (robot description, xacro)
@@ -1,7 +1,4 @@
 <?xml version="1.0"?>
-<robot xmlns:sensor="http://playerstage.sourceforge.net/gazebo/xmlschema/#sensor"
-       xmlns:controller="http://playerstage.sourceforge.net/gazebo/xmlschema/#controller"
-       xmlns:interface="http://playerstage.sourceforge.net/gazebo/xmlschema/#interface"
-       xmlns:xacro="http://ros.org/wiki/xacro">
+<robot xmlns:xacro="http://ros.org/wiki/xacro">
   <!--  Caster wheel transmission   -->
   <xacro:macro name="pr2_wheel_transmission_v0" params="suffix parent reflect">

File: pr2_description/urdf/base_v0/base.urdf.xacro (robot description, xacro)
@@ -1,7 +1,4 @@
 <?xml version="1.0"?>
-<robot xmlns:sensor="http://playerstage.sourceforge.net/gazebo/xmlschema/#sensor"
-       xmlns:controller="http://playerstage.sourceforge.net/gazebo/xmlschema/#controller"
-       xmlns:interface="http://playerstage.sourceforge.net/gazebo/xmlschema/#interface"
-       xmlns:xacro="http://ros.org/wiki/xacro">
+<robot xmlns:xacro="http://ros.org/wiki/xacro">
   <xacro:include filename="$(find pr2_description)/urdf/sensors/hokuyo_lx30_laser.urdf.xacro" />
   <xacro:include filename="$(find pr2_description)/urdf/base_v0/base.gazebo.xacro" />
@@ -11,28 +8,28 @@
   <!-- all link geometry sizes are obtained from Function provided CAD model unless stated otherwise -->
   <!-- all simplified collision geometry are hand approximated from CAD model, sometimes from respective bounding boxes -->
-  <property name="M_PI" value="3.1415926535897931" />
-  <property name="caster_offset_x" value="0.2246" />
-  <property name="caster_offset_y" value="0.2246" />
-  <property name="caster_offset_z" value="0.0282" />
-  <property name="caster_wheel_offset_y" value="0.049" />
-  <property name="wheel_length" value="0.034" />
-  <property name="wheel_radius" value="0.074792" />   <!-- This is the 'effective' wheel radius. Wheel radius for uncompressed wheel is 0.079.  mp 20080801 -->
-  <property name="base_cg_x" value="-0.061" />
-  <property name="base_cg_y" value="0.0" />
-  <property name="base_cg_z" value="${0.5*0.293}" />
-  <property name="base_mass" value="116.0" />
+  <xacro:property name="M_PI" value="3.1415926535897931" />
+  <xacro:property name="caster_offset_x" value="0.2246" />
+  <xacro:property name="caster_offset_y" value="0.2246" />
+  <xacro:property name="caster_offset_z" value="0.0282" />
+  <xacro:property name="caster_wheel_offset_y" value="0.049" />
+  <xacro:property name="wheel_length" value="0.034" />
+  <xacro:property name="wheel_radius" value="0.074792" />   <!-- This is the 'effective' wheel radius. Wheel radius for uncompressed wheel is 0.079.  mp 20080801 -->
+  <xacro:property name="base_cg_x" value="-0.061" />
+  <xacro:property name="base_cg_y" value="0.0" />
+  <xacro:property name="base_cg_z" value="${0.5*0.293}" />
+  <xacro:property name="base_mass" value="116.0" />
   <!-- simplified box collision geometry for base -->
-  <property name="base_size_x" value="0.65" />
-  <property name="base_size_y" value="0.65" />
-  <property name="base_size_z" value="0.23" />
-  <property name="base_collision_size_z" value="0.04" />
+  <xacro:property name="base_size_x" value="0.65" />
+  <xacro:property name="base_size_y" value="0.65" />
+  <xacro:property name="base_size_z" value="0.23" />
+  <xacro:property name="base_collision_size_z" value="0.04" />
   <!-- simplified box collision geometry for hokuyo laser -->
-  <property name="base_laser_x" value="0.275" />
-  <property name="base_laser_y" value="0.0" />
-  <property name="base_laser_z" value="0.252" />
-  <property name="base_laser_size_x" value="0.06" />
-  <property name="base_laser_size_y" value="0.06" />
-  <property name="base_laser_size_z" value="0.03" />
-  <property name="base_laser_collision_offset_z" value="0.023" />
+  <xacro:property name="base_laser_x" value="0.275" />
+  <xacro:property name="base_laser_y" value="0.0" />
+  <xacro:property name="base_laser_z" value="0.252" />
+  <xacro:property name="base_laser_size_x" value="0.06" />
+  <xacro:property name="base_laser_size_y" value="0.06" />
+  <xacro:property name="base_laser_size_z" value="0.03" />
+  <xacro:property name="base_laser_collision_offset_z" value="0.023" />
   <!--                                                      -->
   <!--           wheel                                      -->
@@ -81,5 +78,5 @@
       <calibration rising="${ref_position}" />
       <dynamics damping="1.0" friction="0.0" />
-      <insert_block name="origin" />
+      <xacro:insert_block name="origin" />
       <parent link="${parent}"/>
       <child link="${suffix}_rotation_link" />
@@ -112,5 +109,5 @@
     <xacro:pr2_caster_hub_v0 parent="${parent}" suffix="${suffix}_caster"
                              ref_position="${ref_position}" >
-      <insert_block name="origin" />
+      <xacro:insert_block name="origin" />
     </xacro:pr2_caster_hub_v0>
     <!-- wheel macros -->

File: pr2_description/urdf/common.xacro (robot description, xacro)
@@ -1,60 +1,60 @@
 <?xml version="1.0"?>
-<robot>
-  <property name="M_PI" value="3.1415926535897931" />
-  <property name="VELOCITY_LIMIT_SCALE" value="0.6" />
+<robot xmlns:xacro="http://ros.org/wiki/xacro">
+  <xacro:property name="M_PI" value="3.1415926535897931" />
+  <xacro:property name="VELOCITY_LIMIT_SCALE" value="0.6" />
   <!-- Gear Ratio Corrections: Divide transmission reductions by these factors (Nominally 1)-->
-  <property name="cal_r_shoulder_pan_gearing"   value="1.0" />
-  <property name="cal_r_shoulder_lift_gearing"  value="1.0" />
-  <property name="cal_r_upper_arm_roll_gearing" value="1.0" />
+  <xacro:property name="cal_r_shoulder_pan_gearing"   value="1.0" />
+  <xacro:property name="cal_r_shoulder_lift_gearing"  value="1.0" />
+  <xacro:property name="cal_r_upper_arm_roll_gearing" value="1.0" />
   <!-- ********** Right Arm ********** -->
   <!-- Flag offsets: Add to the optical flag locations (Nominally 0) -->
-  <property name="cal_r_shoulder_pan_flag"   value="0.0" />
-  <property name="cal_r_shoulder_lift_flag"  value="0.0" />
-  <property name="cal_r_upper_arm_roll_flag" value="0.0" />
-  <property name="cal_r_elbow_flex_flag"     value="0.0" />
-  <property name="cal_r_forearm_roll_flag"   value="0.0" />
-  <property name="cal_r_wrist_flex_flag"     value="0.0" />
-  <property name="cal_r_wrist_roll_flag"     value="0.0" />
+  <xacro:property name="cal_r_shoulder_pan_flag"   value="0.0" />
+  <xacro:property name="cal_r_shoulder_lift_flag"  value="0.0" />
+  <xacro:property name="cal_r_upper_arm_roll_flag" value="0.0" />
+  <xacro:property name="cal_r_elbow_flex_flag"     value="0.0" />
+  <xacro:property name="cal_r_forearm_roll_flag"   value="0.0" />
+  <xacro:property name="cal_r_wrist_flex_flag"     value="0.0" />
+  <xacro:property name="cal_r_wrist_roll_flag"     value="0.0" />
   <!-- ********** Head ********** -->
   <!-- Head Location: Add to the transform from torso to head_pan_link (Nominally 0) -->
-  <property name="cal_head_x" value="0.0" />
-  <property name="cal_head_y" value="0.0" />
-  <property name="cal_head_z" value="0.0" />
-  <property name="cal_head_roll" value="0.0" />
-  <property name="cal_head_pitch" value="0.0" />
-  <property name="cal_head_yaw" value="0.0" />
+  <xacro:property name="cal_head_x" value="0.0" />
+  <xacro:property name="cal_head_y" value="0.0" />
+  <xacro:property name="cal_head_z" value="0.0" />
+  <xacro:property name="cal_head_roll" value="0.0" />
+  <xacro:property name="cal_head_pitch" value="0.0" />
+  <xacro:property name="cal_head_yaw" value="0.0" />
   <!-- Flag Offsets -->
-  <property name="cal_head_pan_flag"  value="0.0" />
-  <property name="cal_head_tilt_flag" value="0.0" />
-  <property name="cal_head_pan_flag" value="0.0"/>
-  <property name="cal_head_tilt_flag" value="0.0"/>
+  <xacro:property name="cal_head_pan_flag"  value="0.0" />
+  <xacro:property name="cal_head_tilt_flag" value="0.0" />
+  <xacro:property name="cal_head_pan_flag" value="0.0"/>
+  <xacro:property name="cal_head_tilt_flag" value="0.0"/>
   <!-- Casters -->
-  <property name="cal_caster_fl" value="0.0" />
-  <property name="cal_caster_fr" value="0.0" />
-  <property name="cal_caster_bl" value="0.0" />
-  <property name="cal_caster_br" value="0.0" />
+  <xacro:property name="cal_caster_fl" value="0.0" />
+  <xacro:property name="cal_caster_fr" value="0.0" />
+  <xacro:property name="cal_caster_bl" value="0.0" />
+  <xacro:property name="cal_caster_br" value="0.0" />
   <!-- Stereo Camera Location (Nominally 0) -->
-  <property name="cal_stereo_x" value="0.0" />
-  <property name="cal_stereo_y" value="0.0" />
-  <property name="cal_stereo_z" value="0.0" />
-  <property name="cal_stereo_roll" value="0.0" />
-  <property name="cal_stereo_pitch" value="0.0" />
-  <property name="cal_stereo_yaw" value="0.0" />
+  <xacro:property name="cal_stereo_x" value="0.0" />
+  <xacro:property name="cal_stereo_y" value="0.0" />
+  <xacro:property name="cal_stereo_z" value="0.0" />
+  <xacro:property name="cal_stereo_roll" value="0.0" />
+  <xacro:property name="cal_stereo_pitch" value="0.0" />
+  <xacro:property name="cal_stereo_yaw" value="0.0" />
   <!-- Kinect Camera Location (Nominally 0) -->
-  <property name="cal_kinect_x" value="0.0" />
-  <property name="cal_kinect_y" value="0.0" />
-  <property name="cal_kinect_z" value="0.0" />
-  <property name="cal_kinect_roll" value="0.0" />
-  <property name="cal_kinect_pitch" value="0.0" />
-  <property name="cal_kinect_yaw" value="0.0" />
+  <xacro:property name="cal_kinect_x" value="0.0" />
+  <xacro:property name="cal_kinect_y" value="0.0" />
+  <xacro:property name="cal_kinect_z" value="0.0" />
+  <xacro:property name="cal_kinect_roll" value="0.0" />
+  <xacro:property name="cal_kinect_pitch" value="0.0" />
+  <xacro:property name="cal_kinect_yaw" value="0.0" />
   <!-- HighDef Camera Location (Nominally 0) -->
-  <property name="cal_high_def_x" value="0.0" />
-  <property name="cal_high_def_y" value="0.0" />
-  <property name="cal_high_def_z" value="0.0" />
-  <property name="cal_high_def_roll" value="0.0" />
-  <property name="cal_high_def_pitch" value="0.0" />
-  <property name="cal_high_def_yaw" value="0.0" />
+  <xacro:property name="cal_high_def_x" value="0.0" />
+  <xacro:property name="cal_high_def_y" value="0.0" />
+  <xacro:property name="cal_high_def_z" value="0.0" />
+  <xacro:property name="cal_high_def_roll" value="0.0" />
+  <xacro:property name="cal_high_def_pitch" value="0.0" />
+  <xacro:property name="cal_high_def_yaw" value="0.0" />
   <!-- Throwing in left arm constants to appease the xacro parser -->
-  <property name="cal_l_shoulder_pan_flag" value="0.000000" />
-  <property name="cal_l_wrist_roll_flag" value="0.0" />
+  <xacro:property name="cal_l_shoulder_pan_flag" value="0.000000" />
+  <xacro:property name="cal_l_wrist_roll_flag" value="0.0" />
 </robot>

File: pr2_description/urdf/forearm_v0/forearm.gazebo.xacro (robot description, xacro)
@@ -1,7 +1,4 @@
 <?xml version="1.0"?>
-<robot xmlns:sensor="http://playerstage.sourceforge.net/gazebo/xmlschema/#sensor"
-       xmlns:controller="http://playerstage.sourceforge.net/gazebo/xmlschema/#controller"
-       xmlns:interface="http://playerstage.sourceforge.net/gazebo/xmlschema/#interface"
-       xmlns:xacro="http://ros.org/wiki/xacro">
+<robot xmlns:xacro="http://ros.org/wiki/xacro">
   <xacro:macro name="pr2_forearm_gazebo_v0" params="side">
     <gazebo reference="${side}_forearm_link">

File: pr2_description/urdf/forearm_v0/forearm.transmission.xacro (robot description, xacro)
@@ -1,7 +1,4 @@
 <?xml version="1.0"?>
-<robot xmlns:sensor="http://playerstage.sourceforge.net/gazebo/xmlschema/#sensor"
-       xmlns:controller="http://playerstage.sourceforge.net/gazebo/xmlschema/#controller"
-       xmlns:interface="http://playerstage.sourceforge.net/gazebo/xmlschema/#interface"
-       xmlns:xacro="http://ros.org/wiki/xacro">
+<robot xmlns:xacro="http://ros.org/wiki/xacro">
   <xacro:macro name="pr2_forearm_transmission_v0" params="side">
     <!-- Wrist flex , Wrist roll -->

File: pr2_description/urdf/forearm_v0/forearm.urdf.xacro (robot description, xacro)
@@ -1,8 +1,5 @@
 <?xml version="1.0"?>
 <!-- XML namespaces -->
-<robot xmlns:sensor="http://playerstage.sourceforge.net/gazebo/xmlschema/#sensor"
-       xmlns:controller="http://playerstage.sourceforge.net/gazebo/xmlschema/#controller"
-       xmlns:interface="http://playerstage.sourceforge.net/gazebo/xmlschema/#interface"
-       xmlns:xacro="http://ros.org/wiki/xacro">
+<robot xmlns:xacro="http://ros.org/wiki/xacro">
   <!-- Things that are needed only for Gazebo (not the physical robot).  These include
        sensor and controller plugin specifications -->
@@ -13,5 +10,5 @@
   <xacro:macro name="pr2_forearm_v0" params="side parent reflect *origin">
     <joint name="${side}_forearm_joint" type="fixed">
-      <insert_block name="origin" /> <!-- transform from parent link to this joint frame -->
+      <xacro:insert_block name="origin" /> <!-- transform from parent link to this joint frame -->
       <parent link="${parent}"/>
       <child link="${side}_forearm_link"/>

File: pr2_description/urdf/gripper_v0/gripper.transmission.xacro (robot description, xacro)
@@ -1,8 +1,4 @@
 <?xml version="1.0"?>
-<robot xmlns:sensor="http://playerstage.sourceforge.net/gazebo/xmlschema/#sensor"
-       xmlns:controller="http://playerstage.sourceforge.net/gazebo/xmlschema/#controller"
-       xmlns:joint="http://playerstage.sourceforge.net/gazebo/xmlschema/#slider"
-       xmlns:interface="http://playerstage.sourceforge.net/gazebo/xmlschema/#interface"
-       xmlns:xacro="http://ros.org/wiki/xacro">
+<robot xmlns:xacro="http://ros.org/wiki/xacro">
   <xacro:macro name="pr2_gripper_transmission_v0" params="side screw_reduction gear_ratio theta0 phi0 t0 L0 h a b r">
     <!-- [lr]_gripper_joint is a fictitious joint, used by transmission for controller gap   -->
@@ -42,5 +38,5 @@
       <simulated_actuated_joint name="${side}_gripper_motor_screw_joint"
                                 passive_actuated_joint="${side}_gripper_motor_slider_joint"
-                                simulated_reduction="3141.6"   />
+                                simulated_reduction="314.16"   />
     </transmission>
   </xacro:macro>

File: pr2_description/urdf/gripper_v0/gripper.urdf.xacro (robot description, xacro)
@@ -1,19 +1,15 @@
 <?xml version="1.0"?>
-<robot xmlns:sensor="http://playerstage.sourceforge.net/gazebo/xmlschema/#sensor"
-       xmlns:controller="http://playerstage.sourceforge.net/gazebo/xmlschema/#controller"
-       xmlns:joint="http://playerstage.sourceforge.net/gazebo/xmlschema/#slider"
-       xmlns:interface="http://playerstage.sourceforge.net/gazebo/xmlschema/#interface"
-       xmlns:xacro="http://ros.org/wiki/xacro">
+<robot xmlns:xacro="http://ros.org/wiki/xacro">
   <xacro:include filename="$(find pr2_description)/urdf/gripper_v0/gripper.gazebo.xacro" />
   <xacro:include filename="$(find pr2_description)/urdf/gripper_v0/gripper.transmission.xacro" />
-  <property name="M_PI" value="3.1415926535897931" />
-  <property name="gripper_upper_angle" value="0.548" />
-  <property name="gripper_lower_angle" value="0.00" />
-  <property name="finger_damping"             value="0.02" />
-  <property name="gripper_damping"            value="10.0" />
-  <property name="finger_tip_damping"         value="0.001" />
-  <property name="finger_joint_effort_limit"  value="1000.0" />
-  <property name="finger_to_finger_tip_x"     value="0.09137" />
-  <property name="palm_to_finger_x"           value="0.07691" />
+  <xacro:property name="M_PI" value="3.1415926535897931" />
+  <xacro:property name="gripper_upper_angle" value="0.548" />
+  <xacro:property name="gripper_lower_angle" value="0.00" />
+  <xacro:property name="finger_damping"             value="0.02" />
+  <xacro:property name="gripper_damping"            value="10.0" />
+  <xacro:property name="finger_tip_damping"         value="0.001" />
+  <xacro:property name="finger_joint_effort_limit"  value="1000.0" />
+  <xacro:property name="finger_to_finger_tip_x"     value="0.09137" />
+  <xacro:property name="palm_to_finger_x"           value="0.07691" />
   <xacro:macro name="pr2_finger_limits_v0">
     <!-- limits on passive finger and finger top joints without
@@ -164,5 +160,5 @@
   <xacro:macro name="pr2_gripper_v0" params="side reflect parent *origin gear_ratio screw_reduction theta0 phi0 t0 L0 h a b r">
     <joint name="${side}_gripper_palm_joint" type="fixed">
-      <insert_block name="origin"/>
+      <xacro:insert_block name="origin"/>
       <parent link="${parent}"/>
       <child link="${side}_gripper_palm_link"/>

File: pr2_description/urdf/head_v0/head.gazebo.xacro (robot description, xacro)
@@ -1,7 +1,4 @@
 <?xml version="1.0"?>
-<robot xmlns:sensor="http://playerstage.sourceforge.net/gazebo/xmlschema/#sensor"
-       xmlns:controller="http://playerstage.sourceforge.net/gazebo/xmlschema/#controller"
-       xmlns:interface="http://playerstage.sourceforge.net/gazebo/xmlschema/#interface"
-       xmlns:xacro="http://ros.org/wiki/xacro">
+<robot xmlns:xacro="http://ros.org/wiki/xacro">
   <xacro:macro name="pr2_head_gazebo_v0" params="name">
     <gazebo reference="${name}_plate_frame">

File: pr2_description/urdf/head_v0/head.transmission.xacro (robot description, xacro)
@@ -1,7 +1,4 @@
 <?xml version="1.0"?>
-<robot xmlns:sensor="http://playerstage.sourceforge.net/gazebo/xmlschema/#sensor"
-       xmlns:controller="http://playerstage.sourceforge.net/gazebo/xmlschema/#controller"
-       xmlns:interface="http://playerstage.sourceforge.net/gazebo/xmlschema/#interface"
-       xmlns:xacro="http://ros.org/wiki/xacro">
+<robot xmlns:xacro="http://ros.org/wiki/xacro">
   <xacro:macro name="pr2_head_pan_transmission_v0" params="name">
     <transmission type="pr2_mechanism_model/SimpleTransmission" name="${name}_trans">
