Commit message: Rebase from 'upstream'

File: pr2_description/urdf/head_v0/head.urdf.xacro (robot description, xacro)
@@ -1,10 +1,7 @@
 <?xml version="1.0"?>
-<robot xmlns:sensor="http://playerstage.sourceforge.net/gazebo/xmlschema/#sensor"
-       xmlns:controller="http://playerstage.sourceforge.net/gazebo/xmlschema/#controller"
-       xmlns:interface="http://playerstage.sourceforge.net/gazebo/xmlschema/#interface"
-       xmlns:xacro="http://ros.org/wiki/xacro">
+<robot xmlns:xacro="http://ros.org/wiki/xacro">
   <xacro:include filename="$(find pr2_description)/urdf/head_v0/head.gazebo.xacro" />
   <xacro:include filename="$(find pr2_description)/urdf/head_v0/head.transmission.xacro" />
-  <property name="M_PI" value="3.1415926535897931" />
+  <xacro:property name="M_PI" value="3.1415926535897931" />
   <xacro:macro name="pr2_head_pan_v0" params="name parent *origin">
     <joint name="${name}_joint" type="revolute">
@@ -14,5 +11,5 @@
       <calibration rising="0.0" />
       <dynamics damping="0.5" />
-      <insert_block name="origin" />
+      <xacro:insert_block name="origin" />
       <parent link="${parent}"/>
       <child link="${name}_link"/>
@@ -48,5 +45,5 @@
       <calibration falling="${0.0+cal_head_tilt_flag}" />
       <dynamics damping="10.0" />
-      <insert_block name="origin" />
+      <xacro:insert_block name="origin" />
       <parent link="${parent}"/>
       <child link="${name}_link"/>
@@ -79,5 +76,5 @@
   <xacro:macro name="pr2_head_v0" params="name parent *origin">
     <xacro:pr2_head_pan_v0 name="${name}_pan" parent="${parent}">
-      <insert_block name="origin" />
+      <xacro:insert_block name="origin" />
     </xacro:pr2_head_pan_v0>
     <xacro:pr2_head_tilt_v0 name="${name}_tilt" parent="${name}_pan_link">

File: pr2_description/urdf/sensors/double_stereo_camera.gazebo.xacro (robot description, xacro)
@@ -1,7 +1,4 @@
 <?xml version="1.0"?>
-<robot xmlns:sensor="http://playerstage.sourceforge.net/gazebo/xmlschema/#sensor"
-       xmlns:controller="http://playerstage.sourceforge.net/gazebo/xmlschema/#controller"
-       xmlns:interface="http://playerstage.sourceforge.net/gazebo/xmlschema/#interface"
-       xmlns:xacro="http://ros.org/wiki/xacro">
+<robot xmlns:xacro="http://ros.org/wiki/xacro">
   <!-- Made by Kevin for double stereo camera for PR-2 Beta. -->
   <!-- Needs calibration verification, and CAD check. -->

File: pr2_description/urdf/sensors/double_stereo_camera.urdf.xacro (robot description, xacro)
@@ -1,14 +1,11 @@
 <?xml version="1.0"?>
-<robot xmlns:sensor="http://playerstage.sourceforge.net/gazebo/xmlschema/#sensor"
-       xmlns:controller="http://playerstage.sourceforge.net/gazebo/xmlschema/#controller"
-       xmlns:interface="http://playerstage.sourceforge.net/gazebo/xmlschema/#interface"
-       xmlns:xacro="http://ros.org/wiki/xacro">
+<robot xmlns:xacro="http://ros.org/wiki/xacro">
   <xacro:include filename="$(find pr2_description)/urdf/sensors/double_stereo_camera.gazebo.xacro" />
   <xacro:include filename="$(find pr2_description)/urdf/sensors/stereo_camera.urdf.xacro" />
-  <property name="stereo_size_x" value="0.02" />
-  <property name="stereo_size_y" value="0.12" />
-  <property name="stereo_size_z" value="0.05" />
-  <property name="stereo_center_box_center_offset_x" value="-0.01" />
-  <property name="stereo_center_box_center_offset_z" value="0.025" />
+  <xacro:property name="stereo_size_x" value="0.02" />
+  <xacro:property name="stereo_size_y" value="0.12" />
+  <xacro:property name="stereo_size_z" value="0.05" />
+  <xacro:property name="stereo_center_box_center_offset_x" value="-0.01" />
+  <xacro:property name="stereo_center_box_center_offset_z" value="0.025" />
   <!-- Made by Kevin for double stereo camera for PR-2 Beta. -->
   <!-- Needs calibration verification, and CAD check. -->
@@ -16,5 +13,5 @@
     <!-- Define link to stereo cameras, set origin relative to that -->
     <joint name="${name}_frame_joint" type="fixed">
-      <insert_block name="origin" />
+      <xacro:insert_block name="origin" />
       <parent link="${parent}"/>
       <child link="${name}_link"/>

File: pr2_description/urdf/sensors/head_sensor_package.gazebo.xacro (robot description, xacro)
@@ -1,8 +1,5 @@
 <?xml version="1.0"?>
-<robot xmlns:sensor="http://playerstage.sourceforge.net/gazebo/xmlschema/#sensor"
-       xmlns:controller="http://playerstage.sourceforge.net/gazebo/xmlschema/#controller"
-       xmlns:interface="http://playerstage.sourceforge.net/gazebo/xmlschema/#interface"
-       xmlns:xacro="http://ros.org/wiki/xacro">
-  <property name="M_PI" value="3.1415926535897931" />
+<robot xmlns:xacro="http://ros.org/wiki/xacro">
+  <xacro:property name="M_PI" value="3.1415926535897931" />
   <!-- Made by Kevin for A2 sensor package -->
   <!-- Origin is center mount screw on sensor plate mount -->

File: pr2_description/urdf/sensors/head_sensor_package.urdf.xacro (robot description, xacro)
@@ -1,7 +1,4 @@
 <?xml version="1.0"?>
-<robot xmlns:sensor="http://playerstage.sourceforge.net/gazebo/xmlschema/#sensor"
-       xmlns:controller="http://playerstage.sourceforge.net/gazebo/xmlschema/#controller"
-       xmlns:interface="http://playerstage.sourceforge.net/gazebo/xmlschema/#interface"
-       xmlns:xacro="http://ros.org/wiki/xacro">
+<robot xmlns:xacro="http://ros.org/wiki/xacro">
   <!-- This urdf macro defines following sensors:
        prosilica
@@ -16,5 +13,5 @@
   <xacro:macro name="pr2_head_sensor_package_v0" params="name hd_frame_name hd_camera_name stereo_name parent *origin">
     <joint name="${name}_frame_joint" type="fixed">
-      <insert_block name="origin" />
+      <xacro:insert_block name="origin" />
       <parent link="${parent}"/>
       <child link="${name}_link"/>

File: pr2_description/urdf/sensors/hokuyo_lx30_laser.urdf.xacro (robot description, xacro)
@@ -1,12 +1,9 @@
 <?xml version="1.0"?>
-<robot xmlns:sensor="http://playerstage.sourceforge.net/gazebo/xmlschema/#sensor"
-       xmlns:controller="http://playerstage.sourceforge.net/gazebo/xmlschema/#controller"
-       xmlns:interface="http://playerstage.sourceforge.net/gazebo/xmlschema/#interface"
-       xmlns:xacro="http://ros.org/wiki/xacro">
+<robot xmlns:xacro="http://ros.org/wiki/xacro">
   <xacro:include filename="$(find pr2_description)/urdf/sensors/hokuyo_lx30_laser.gazebo.xacro" />
   <xacro:macro name="hokuyo_lx30_laser_v0" params="name parent *origin ros_topic update_rate min_angle max_angle">
     <joint name="${name}_joint" type="fixed">
       <axis xyz="0 1 0" />
-      <insert_block name="origin" />
+      <xacro:insert_block name="origin" />
       <parent link="${parent}_link"/>
       <child link="${name}_link"/>

Commit message: Rebase from 'upstream'

File: pr2_description/robots/pr2.urdf.xacro (robot description, xacro)
@@ -1,8 +1,4 @@
 <?xml version="1.0"?>
-<robot xmlns:sensor="http://playerstage.sourceforge.net/gazebo/xmlschema/#sensor"
-       xmlns:controller="http://playerstage.sourceforge.net/gazebo/xmlschema/#controller"
-       xmlns:interface="http://playerstage.sourceforge.net/gazebo/xmlschema/#interface"
-       xmlns:xacro="http://playerstage.sourceforge.net/gazebo/xmlschema/#interface"
-       name="pr2" >
+<robot xmlns:xacro="http://ros.org/wiki/xacro" name="pr2" >
   <!-- The following included files set up definitions of parts of the robot body -->
   <!-- misc common stuff? -->
@@ -24,5 +20,4 @@
   <!-- Head sensors -->
   <xacro:include filename="$(find pr2_description)/urdf/sensors/head_sensor_package.urdf.xacro" />
-  <xacro:include filename="$(find pr2_description)/urdf/sensors/kinect_prosilica_camera.urdf.xacro" />
   <!-- Camera sensors -->
   <xacro:include filename="$(find pr2_description)/urdf/sensors/wge100_camera.urdf.xacro" />
@@ -63,20 +58,4 @@
     <origin xyz="0 0.110 0.0546" rpy="0 0 0" />
   </xacro:projector_wg6802418_v0>
-  <!-- Base of Kinect/Prosilica Mount -->
-  <xacro:kinect_prosilica_camera_swept_back_v0 name="head_mount" parent="head_plate_frame" >
-    <origin xyz="-0.137376 0 0.091746" rpy="0 0 0" />
-    <!--
-          Was -0.1 0 0.09225, -0.138 0 0.09225 looks good front back and sheet metal on bolt pattern,
-          -0.138 0 0.06225 is where Prosilica FOV just clears the head.
-          This is 30 mm (!) below the position in SolidWorks.
-          Lowering the Prosilica by this amount in SW makes the FOV hit around the aluminum / plastic junction.
-          Turns out that head_plate_frame is in some random position in space.
-          It is [0.0232 0 0.0645 from its parent, head_tilt_link.
-          The distance from head_plate_frame to the head_kinect_prosilica is 137.376 mm X and 91.746 mm Z.
-          So the origin should in fact be -0.137376 0 0.091746.
-          John is changing the Prosilica FOV based on my numbers.
-          Just need to roscd and svn up.
-    -->
-  </xacro:kinect_prosilica_camera_swept_back_v0>
   <xacro:pr2_tilting_laser_v0 name="laser_tilt" parent="torso_lift_link" laser_calib_ref="0.0">
     <origin xyz="0.09893 0 0.227" rpy="0 0 0" />
@@ -139,3 +118,35 @@
     <origin xyz=".135 0 .044" rpy="${M_PI/2} ${-32.25*M_PI/180} 0" />
   </xacro:wge100_camera_v0>
+  <!-- Kinect models -->
+  <xacro:arg name="KINECT1" default="false" />
+  <xacro:arg name="KINECT2" default="false" />
+  <!-- Kinect2 xacro -->
+  <xacro:if value="$(arg KINECT2)">
+    <xacro:include filename="$(find pr2_description)/urdf/sensors/kinect2.urdf.xacro" />
+    <xacro:kinect2_v0 name="head_mount" parent="head_plate_frame" >
+      <origin xyz="-0.137376 0 0.091746" rpy="0 0 0" />
+    </xacro:kinect2_v0>
+  </xacro:if>
+  <!-- Kinect1 xacro -->
+  <xacro:unless value="$(arg KINECT2)">
+    <xacro:if value="$(arg KINECT1)">
+      <xacro:include filename="$(find pr2_description)/urdf/sensors/kinect_prosilica_camera.urdf.xacro" />
+      <!-- Base of Kinect/Prosilica Mount -->
+      <xacro:kinect_prosilica_camera_swept_back_v0 name="head_mount" parent="head_plate_frame" >
+        <origin xyz="-0.137376 0 0.091746" rpy="0 0 0" />
+        <!--
+              Was -0.1 0 0.09225, -0.138 0 0.09225 looks good front back and sheet metal on bolt pattern,
+              -0.138 0 0.06225 is where Prosilica FOV just clears the head.
+              This is 30 mm (!) below the position in SolidWorks.
+              Lowering the Prosilica by this amount in SW makes the FOV hit around the aluminum / plastic junction.
+              Turns out that head_plate_frame is in some random position in space.
+              It is [0.0232 0 0.0645 from its parent, head_tilt_link.
+              The distance from head_plate_frame to the head_kinect_prosilica is 137.376 mm X and 91.746 mm Z.
+              So the origin should in fact be -0.137376 0 0.091746.
+              John is changing the Prosilica FOV based on my numbers.
+              Just need to roscd and svn up.
+        -->
+      </xacro:kinect_prosilica_camera_swept_back_v0>
+    </xacro:if>
+  </xacro:unless>
 </robot>

File: pr2_description/urdf/sensors/kinect_camera.urdf.xacro (robot description, xacro)
@@ -1,11 +1,8 @@
 <?xml version="1.0"?>
-<root xmlns:sensor="http://playerstage.sourceforge.net/gazebo/xmlschema/#sensor"
-      xmlns:controller="http://playerstage.sourceforge.net/gazebo/xmlschema/#controller"
-      xmlns:interface="http://playerstage.sourceforge.net/gazebo/xmlschema/#interface"
-      xmlns:xacro="http://ros.org/wiki/xacro">
+<robot xmlns:xacro="http://ros.org/wiki/xacro">
   <xacro:include filename="$(find pr2_description)/urdf/sensors/kinect_camera.gazebo.xacro" />
   <xacro:macro name="kinect_camera_v0" params="name parent *origin">
     <joint name="${name}_frame_joint" type="fixed">
-      <insert_block name="origin" />
+      <xacro:insert_block name="origin" />
       <parent link="${parent}"/>
       <child link="${name}_frame"/>
@@ -42,3 +39,3 @@
     <xacro:kinect_camera_gazebo_v0 name="${name}" />
   </xacro:macro>
-</root>
+</robot>

File: pr2_description/urdf/sensors/kinect_prosilica_camera.gazebo.xacro (robot description, xacro)
@@ -23,6 +23,6 @@
         <updateRate>1.0</updateRate>
         <cameraName>${camera_name}_ir</cameraName>
-        <imageTopicName>/${camera_name}/depth/image_raw</imageTopicName>
-        <cameraInfoTopicName>/${camera_name}/depth/camera_info</cameraInfoTopicName>
+        <imageTopicName>/${camera_name}/ir/image_raw</imageTopicName>
+        <cameraInfoTopicName>/${camera_name}/ir/camera_info</cameraInfoTopicName>
         <depthImageTopicName>/${camera_name}/depth/image_raw</depthImageTopicName>
         <depthImageCameraInfoTopicName>/${camera_name}/depth/camera_info</depthImageCameraInfoTopicName>
@@ -53,5 +53,5 @@
         <horizontal_fov>${57.0*M_PI/180.0}</horizontal_fov>
         <image>
-          <format>R8G8B8</format>
+          <format>B8G8R8</format>
           <width>640</width>
           <height>480</height>

File: pr2_description/urdf/sensors/kinect_prosilica_camera.urdf.xacro (robot description, xacro)
@@ -1,9 +1,6 @@
 <?xml version="1.0"?>
-<root xmlns:sensor="http://playerstage.sourceforge.net/gazebo/xmlschema/#sensor"
-      xmlns:controller="http://playerstage.sourceforge.net/gazebo/xmlschema/#controller"
-      xmlns:interface="http://playerstage.sourceforge.net/gazebo/xmlschema/#interface"
-      xmlns:xacro="http://ros.org/wiki/xacro">
+<root xmlns:xacro="http://ros.org/wiki/xacro">
   <xacro:include filename="$(find pr2_description)/urdf/sensors/kinect_prosilica_camera.gazebo.xacro" />
-  <property name="ir_depth_rgb_offset_y" value="0.01"/> <!-- FIXME: what is this offset? -->
+  <xacro:property name="ir_depth_rgb_offset_y" value="0.01"/> <!-- FIXME: what is this offset? -->
   <!-- kinect and prosilica combo -->
   <xacro:macro name="kinect_prosilica_camera_swept_back_v0" params="name parent *origin">
@@ -11,5 +8,5 @@
     <joint name="${name}_joint" type="fixed">
       <!-- <limit lower="0.1" upper="0.1" effort="10000" velocity="100.0"/> -->
-      <!-- <insert_block name="origin" /> -->
+      <!-- <xacro:insert_block name="origin" /> -->
       <origin xyz="-0.138 0 0.091" rpy="0 0 0"/>
       <parent link="${parent}"/>

File: pr2_description/urdf/upper_arm_v0/upper_arm.gazebo.xacro (robot description, xacro)
@@ -1,7 +1,4 @@
 <?xml version="1.0"?>
-<robot xmlns:sensor="http://playerstage.sourceforge.net/gazebo/xmlschema/#sensor"
-       xmlns:controller="http://playerstage.sourceforge.net/gazebo/xmlschema/#controller"
-       xmlns:interface="http://playerstage.sourceforge.net/gazebo/xmlschema/#interface"
-       xmlns:xacro="http://ros.org/wiki/xacro">
+<robot xmlns:xacro="http://ros.org/wiki/xacro">
   <xacro:macro name="pr2_upper_arm_gazebo_v0" params="side">
     <gazebo reference="${side}_upper_arm_link">
@@ -11,8 +8,9 @@
   <!-- Elbow flex -->
   <xacro:macro name="pr2_elbow_flex_gazebo_v0" params="side">
-    <!-- testing initial joint position, to be parsed at urdf2gazebo parse time -->
+    <!-- testing initial joint position, to be parsed at urdf2gazebo parse time ->
     <gazebo reference="${side}_elbow_flex_joint">
       <initial_joint_position>-1.0</initial_joint_position>
     </gazebo>
+    -->
     <gazebo reference="${side}_elbow_flex_link">
       <turnGravityOff>true</turnGravityOff>
