Commit message: Imported upstream version '1.13.0' of 'upstream'

File: pr2_description/urdf/sensors/kinect2.urdf.xacro (robot description, xacro)
@@ -21,5 +21,5 @@
         <origin xyz="-0.102 -0.148 0" rpy="0 0 0"/>
         <geometry>
-          <mesh filename="package://pr2_description/meshes/sensors/kinect2_v0/kinect2_assembly.STL" scale="0.001 0.001 0.001" />
+          <mesh filename="package://pr2_description/meshes/sensors/kinect2_v0/kinect2_assembly.dae" scale="0.001 0.001 0.001" />
         </geometry>
         <material name="gray">
@@ -28,7 +28,7 @@
       </visual>
       <collision>
-        <origin xyz="0 0 0" rpy="0 0 0"/>
+        <origin xyz="-0.042 0 0.1" rpy="0 0 0"/>
         <geometry>
-          <sphere radius="0.0005"/>
+          <box size="0.12 0.3 0.2"/>
         </geometry>
       </collision>
@@ -48,16 +48,4 @@
                  izz="0.01" />
       </inertial>
-      <visual>
-        <origin xyz="0.0 0.0 0" rpy="0 0 0"/>
-        <geometry>
-          <sphere radius="0.0005"/>
-        </geometry>
-      </visual>
-      <collision>
-        <origin xyz="0.0 0.0 0" rpy="0 0 0"/>
-        <geometry>
-          <sphere radius="0.0005"/>
-        </geometry>
-      </collision>
     </link>
     <!-- kinect2 ir sensor frame -->
@@ -85,17 +73,4 @@
                  izz="0.01" />
       </inertial>
-      <visual>
-        <origin xyz="${cal_kinect_x}            ${cal_kinect_y}                 ${cal_kinect_z}"
-                rpy="${-M_PI/2+cal_kinect_roll} ${0.0+cal_kinect_pitch}         ${-M_PI/2+cal_kinect_yaw}" />
-        <geometry>
-          <sphere radius="0.0005"/>
-        </geometry>
-      </visual>
-      <collision>
-        <origin xyz="0.0 0.0 0" rpy="0 0 0"/>
-        <geometry>
-          <sphere radius="0.0005"/>
-        </geometry>
-      </collision>
     </link>
     <!-- kinect2 rgb sensor frame -->
